File: PCB/TwinPanda.kicad_pcb (KiCad board)
At the start: 2 copper layers, 407.6 x 180.4 mm, 194 parts, among them J2 Conn_01x04_Socket, SW1 4-0, SW10 4-4, SW11 t2-0, SW12 T2-0, SW13 t2-1, SW14 T2-1, SW15 3-0, SW16 3-1, SW17 3-2, SW18 3-3, SW19 3-4, SW2 4-0, SW20 3-5, SW21 3-6, SW22 3-0, SW23 3-1, SW24 3-2, SW25 3-3, SW26 3-4, SW27 3-5, SW28 3-6, SW29 2-0, SW3 4-1, SW30 2-1, SW31 2-2, SW32 2-3, SW33 2-4, SW34 2-5, SW35 t0-1, SW36 2-0, SW37 2-1, SW38 2-2, SW39 2-3, SW4 4-1, SW40 2-4, SW41 2-5, SW42 T0-1, SW43 1-0, SW44 1-1, SW45 1-2, SW46 1-3, SW47 1-4, SW48 1-5, SW49 1-6, SW5 4-2, SW50 1-0, SW51 1-1, SW52 1-2, SW53 1-3, SW54 1-4, SW55 1-5, SW56 1-6, SW57 0-0, SW58 0-1, SW59 0-2, SW6 4-2, SW60 0-3, SW61 0-4, SW62 0-5, SW63 0-6, SW64 0-0, SW65 0-1, SW66 0-2, SW67 0-3, SW68 0-4, SW69 0-5, SW7 4-3, SW70 0-6, SW71 RotaryEncoder_Switch, SW72 t0-2, SW73 t1-2, SW74 t2-2, SW75 RotaryEncoder_Switch, SW77 T0-2, SW78 T1-2, SW79 T2-2, SW8 4-3, SW9 4-4, U2 XIAO-nRF52840-SMD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

Commit message: Update BOM, PCB layout, and assembly images
Updated BOM.csv with new suppliers, lower prices, and alternative links for several components. Modified the PCB layout (TwinPanda.kicad_pcb) with significant changes to component and mounting hole positions. Refreshed FullAssembly.png and PCB.png images to reflect the latest design.
Parts:
- moved D41 219.1 mm to (478.4, 223.0)
- moved D73 219.1 mm to (485.5, 249.2)
- moved SW72 219.1 mm to (488.3, 226.0)
- moved TP3 219.1 mm to (490.5, 142.0)
- moved U2 219.1 mm to (479.6, 115.1)
- moved D11 219.1 mm to (442.2, 142.5)
- moved D17 219.1 mm to (442.2, 161.6)
- moved D19 219.1 mm to (423.1, 161.6)
- moved D37 219.1 mm to (423.1, 180.6)
- moved D39 219.1 mm to (442.2, 180.6)
- moved D45 219.1 mm to (442.2, 199.7)
- moved D47 219.1 mm to (423.1, 199.7)
- moved D57 219.1 mm to (346.9, 218.7)
- moved D65 219.1 mm to (423.1, 214.0)
- moved D67 219.1 mm to (445.2, 243.0)
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Other:
- board size 407.6 x 180.4 mm -> 391.8 x 180.4 mm
